File: esp-eval/esp-eval.kicad_pcb (KiCad board)
At the start: 2 copper layers, 26 parts, among them J1 ESP-ADAPT-1, J10 ESP-ADAPT-2-SHIELD, J2 ESP-ADAPT-2, J3 ESP-ADAPT-1-DBG, J4 ESP-ADAPT-2-DBG, J5 GPIO0-SEL, J6 GPIO2-SEL, J7 GPIO15-SEL, J8 USB-FTDI, J9 ESP-ADAPT-1-SHIELD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

Commit message: pcb rule check
Parts:
- moved J10 1.38 mm to (28.6, 21.8)
- moved J9 1.38 mm to (28.9, 51.9)
- moved U2 1.38 mm to (57.0, 32.5)
Routing:
- net /esp-12-adapt/VCC: track 19.2 -> 21.1 mm
- net /esp-12-adapt/SCLK: track 10.0 -> 11.1 mm
- net /esp-12-adapt/GPIO9: track 16.4 -> 17.1 mm
